File: HABBoard/HABBoard.kicad_sch (KiCad schematic)
At the start: 64 parts

Commit message: Added GPS Module
Parts:
- added C?: 0.1u, symbol Device:C_Small
- added J?: GPS_SMA, symbol Connector:Conn_Coaxial
- added L?: 27n, symbol Device:L_Small
- added R?: 22, symbol Device:R_Small
- added TP?: GNSS_RESET, symbol Connector:TestPoint
- added TP?: GNSS_SB, symbol Connector:TestPoint
- added U?: NEO-M9N-00B, HABParts:XCVR_NEO-M9N-00B, symbol HABParts:NEO-M9N-00B
Connections:
- net +3V3: now also U?.23 (VCC)
- net GND: now also C?.2, J?.2 (Ext), U?.10 (GND), U?.12 (GND), U?.13 (GND), U?.24 (GND), U?.7 (V_USB)
- new net: C?.1, L?.1, R?.1
- new net: J?.1 (In), L?.2, U?.11 (RF_IN)
- new net: TP?.1, U?.8 (RESET_N)
- new net: TP?.1, U?.1 (SAFEBOOT_N)
- new net: U?.15 (RESERVED), U?.16 (RESERVED), U?.17 (RESERVED)
- new net: R?.2, U?.9 (VCC_RF)
- new net GNSS_SCL: U?.19 (SCL/SPI_CLK)
- new net GNSS_SDA: U?.18 (SDA/SPI_CS_N)
- no-connect marks 4 -> 9
Other:
- moved on the sheet: BT?, C?, D?, J?, L?, Q?A, Q?B, R?, SW?, TH?, U?

Commit message: Revisions before battery change
Parts:
- added C? (x2): 0.1u, symbol Device:C_Small
- added C? (x2): 2.2u, symbol Device:C_Small
- added U?: BMP581, HABParts:BMP581, symbol HABParts:BMP581
- added U?: AP2138N-2.5, Package_TO_SOT_SMD:SOT-23, symbol HABParts:AP2138N-2.5
Connections:
- net +3V3: now also C?.1, C?.1, U?.1 (VDDIO), U?.10 (VDD), U?.5 (SDO/ADR), U?.6 (CSB)
- net +SYS: now also C?.2, U?.3 (VIN)
- net GND: now also C?.1, C?.2, C?.2, C?.2, U?.1 (GND), U?.3 (GND), U?.8 (GND), U?.9 (GND)
- net at U?.22 (V_BCKP): now also C?.1, U?.2 (VOUT)
- new net BRM_INT: U?.7 (INT)
- new net BRM_SCL: U?.2 (SCK/SCL)
- new net BRM_SDA: U?.4 (SDI/SDA)
Other:
- moved on the sheet: C?, J?, L?, R?, TP?, U?

Commit message: Added the rest of the sensors
Parts:
- removed BT?: BATT, symbol Device:Battery_Cell
- removed C? (x4): 0.1u, symbol Device:C_Small
- removed C? (x3): 10u, symbol Device:C_Small
- removed C?: 0.47u, symbol Device:C_Small
- removed C? (x3): 2.2u, symbol Device:C_Small
- removed C?: 22u, symbol Device:C_Small
- removed D?: STAT, symbol Device:LED_Small
- removed J?: USB, symbol Connector:USB_C_Receptacle_USB2.0
- removed L?: 0.47u, symbol Device:L_Small
- removed Q? (x2): PMDPB30XN, HABParts:DMN1025UFDB7, symbol HABParts:PMDPB30XN
- removed R?: Rled, symbol Device:R_Small
- removed R?: 100, symbol Device:R_Small
- removed R?: 22, symbol Device:R_Small
- removed R?: 200K, symbol Device:R_Small
- removed R?: Rthm, symbol Device:R_Small
- removed R?: 1K, symbol Device:R_Small
- removed R?: 18.7K, symbol Device:R_Small
- removed R?: 10m, symbol Device:R_Small
- removed R?: 2.26m, symbol Device:R_Small
- removed TH?: THM, symbol Device:Thermistor_NTC
- removed TP?: GNSS_RESET, symbol Connector:TestPoint
- removed U?: TC7USB40FT, Package_SO:TSSOP-14_4.4x5mm_P0.65mm, symbol HABParts:TC7USB40FT
- removed U?: MAX77757JEFG420+, HABParts:IC_MAX77757JEFG420+, symbol HABParts:MAX77757JEFG420+
- removed U?: bq298215, symbol HABParts:bq298215
- removed U?: MAX17260SETD, Package_DFN_QFN:TDFN-14-1EP_3x3mm_P0.4mm_EP1.78x2.35mm, symbol HABParts:MAX17260SETD
- added C? (x2): 2.2u, symbol Device:C_Small
- added C? (x5): 0.1u, symbol Device:C_Small
- added R? (x2): 2.2K, symbol Device:R_Small
- added R? (x2): 10K (DNF), symbol Device:R_Small
- added SW?: RESET, symbol Switch:SW_Push
- added U?: AP2138N-1.8, Package_TO_SOT_SMD:SOT-23, symbol HABParts:AP2138N-1.8
- added U?: ADT7410TRZ, SOIC127P600X175-8N_ADT7410TRZ, symbol HABParts:ADT7410TRZ
- added U?: Si4063, Package_DFN_QFN:QFN-20-1EP_4x4mm_P0.5mm_EP2.6x2.6mm_ThermalVias, symbol HABParts:Si4063
- added U?: ICM-20948, Sensor_Motion:InvenSense_QFN-24_3x3mm_P0.4mm, symbol Sensor_Motion:ICM-20948
- added U?: TXS0104E, Package_SO:TSSOP-14_4.4x5mm_P0.65mm, symbol HABParts:TXS0104E
Connections:
- net MCU_DN is gone; now on an unnamed net: U?.46 (USB_DM)
- net MCU_DP is gone; now on an unnamed net: U?.47 (USB_DP)
- net +3V3: now also C?.1, C?.1, C?.2, R?.2, R?.2, U?.14 (VCCB), U?.3 (VIN), U?.6 (VDD), U?.8 (VDD), U?.8 (VDD)
- net GND: now also C?.1, C?.2, C?.2, C?.2, C?.2, C?.2, C?.2, SW?.1, U?.1 (GND), U?.18 (GND), U?.18 (GND), U?.20 (GND), U?.21 (GND), U?.3 (A0), U?.4 (A1), U?.7 (GND), U?.7 (GND)
- net at U?.8 (RESET_N): now also SW?.2
- new net: C?.1, U?.10 (REGOUT)
- new net: R?.1, U?.5 (INT)
- new net: R?.1, U?.6 (CT)
- new net: R?.1, U?.2 (A1), U?.24 (SDA/SDI)
- new net: R?.1, U?.23 (SCL/SCLK), U?.3 (A2)
- new net: U?.12 (INT1), U?.4 (A3)
- new net +1V8: C?.1, C?.1, C?.1, R?.2, R?.2, U?.1 (VCCA), U?.13 (VDD), U?.2 (VOUT), U?.22 (~{CS}), U?.8 (OE), U?.8 (VDDIO)
- new net IMU_INT: U?.12 (B3)
- new net IMU_SCL: U?.11 (B2)
- new net IMU_SDA: U?.10 (B1)
- new net TMP_SCL: U?.1 (SCL)
- new net TMP_SDA: U?.2 (SDA)
- no-connect marks 9 -> 11
Other:
- moved on the sheet: C?, J?, L?, R?, SW?, TP?, U?

Commit message: RF Analog Design
Parts:
- removed U?: Si4063, Package_DFN_QFN:QFN-20-1EP_4x4mm_P0.5mm_EP2.6x2.6mm_ThermalVias, symbol HABParts:Si4063
- added BT?: Battery, symbol Device:Battery
- added C?: 22p, symbol Device:C_Small
- added C?: 39p, symbol Device:C_Small
- added C? (x2): 10n, symbol Device:C_Small
- added C? (x2): 1u, symbol Device:C_Small
- added C?: 1.5p, symbol Device:C_Small
- added C? (x6): 47p, symbol Device:C_Small
- added C?: 4.7p, symbol Device:C_Small
- added C? (x3): 100p, symbol Device:C_Small
- added C? (x2): 27p, symbol Device:C_Small
- added C? (x2): 8.2p, symbol Device:C_Small
- added C? (x2): 3.3p, symbol Device:C_Small
- added J?: 144MHz, symbol Connector:Conn_Coaxial
- added J?: 915MHz, symbol Connector:Conn_Coaxial
- added L?: 100n, symbol Device:L_Small
- added L? (x3): 39n, symbol Device:L_Small
- added L?: 4.7n, symbol Device:L_Small
- added L?: 5.6n, symbol Device:L_Small
- added L?: 10n, symbol Device:L_Small
- added L?: 2.2n, symbol Device:L_Small
- added L?: 33n, symbol Device:L_Small
- added Q?: PMN16XNE, Package_SO:TSOP-6_1.65x3.05mm_P0.95mm, symbol HABParts:PMN16XNE
- added R?: 300K, symbol Device:R_Small
- added R?: 120K, symbol Device:R_Small
- added R?: 680, symbol Device:R_Small
- added U? (x2): SX1276, Package_DFN_QFN:QFN-28-1EP_6x6mm_P0.65mm_EP4.8x4.8mm, symbol RF:SX1276
- added U?: MP5016GQH-Z, HABParts:IC_MP5016GQH-Z, symbol HABParts:MP5016GQH-Z
- added U?: PE42421, Package_TO_SOT_SMD:SOT-363_SC-70-6, symbol HABParts:PE42421
- R?: value 10K (DNF) -> 10K
Connections:
- net +SYS: now also C?.1, Q?.4 (S)
- net GND: now also BT?.2 (-), C?.2, C?.2, C?.2, C?.2, C?.2, C?.2, C?.2, C?.2, C?.2, C?.2, C?.2, C?.2, C?.2, C?.2, C?.2, C?.2, C?.2, J?.2 (Ext), J?.2 (Ext), R?.1, R?.1, U?.15 (GND), U?.15 (GND), U?.2 (GND), U?.23 (GND), U?.23 (GND), U?.26 (GND), U?.26 (GND), U?.29 (GND), U?.29 (GND), U?.3 (GND)
- net TMP_INT: now reaches R?.1, U?.5 (INT)
- new net: C?.1, C?.1, L?.2, L?.2
- new net: C?.2, L?.1 (x2)
- new net: C?.1, C?.1, C?.1, L?.1, U?.25 (VR_PA) (x2)
- new net: C?.1, C?.1, L?.2, U?.27 (PA_BOOST)
- new net: C?.1, C?.1, L?.1, L?.2 (x2)
- new net: C?.1, R?.2, U?.5 (MODE)
- new net: C?.1, J?.1 (In), L?.2
- new net: U?.20 (RXTX/RF_MOD), U?.4 (CRTL)
- new net: L?.1, U?.21 (RFI_HF)
- new net: L?.1, U?.27 (PA_BOOST)
- new net: C?.2, J?.1 (In)
- new net: C?.1, C?.2, L?.2, U?.3 (RF2)
- new net: R?.1, U?.9 (EN)
- new net: BT?.1 (+), C?.1, R?.2, U?.1 (VCC), U?.2 (VCC)
- new net: Q?.1 (D), Q?.2 (D), Q?.5 (D), Q?.6 (D), U?.6 (SOURCE), U?.7 (SOURCE)
- new net: Q?.3 (G), U?.8 (GATE)
- new net: C?.1, C?.2, L?.1, L?.2
- new net: R?.2, U?.4 (ILMIT)
- new net: C?.2, U?.1 (RF1)
- new net: C?.1, U?.5 (RFC)
- new net: C?.1, C?.1, L?.2
- no-connect marks 11 -> 20
Other:
- moved on the sheet: C?, L?, SW?, U?

Commit message: More RF Stuff
Parts:
- added C? (x11): 0.1u, symbol Device:C_Small
- added C?: C, symbol Device:C_Small
- added J? (x2): RFShield_TwoPieces, symbol Device:RFShield_TwoPieces
- added R? (x2): R, symbol Device:R_Small
- added R?: 27m, symbol Device:R_Small
- added RN? (x4): 100, symbol Device:R_Pack04
- added U?: INA219BxD, Package_SO:SOIC-8_3.9x4.9mm_P1.27mm, symbol Analog_ADC:INA219BxD
Connections:
- net +3V3: now also U?.14 (VBAT_DIG), U?.14 (VBAT_DIG), U?.24 (VBAT_RF), U?.24 (VBAT_RF), U?.3 (VBAT_ANA), U?.3 (VBAT_ANA), C?.1, C?.1, C?.1, C?.1, C?.1, C?.1, C?.1, U?.5 (VS)
- net +SYS: now also R?.1, R?.1; no longer C?.1, Q?.4 (S)
- net GND: now also C?.2, C?.2, C?.2, C?.2, C?.2, C?.2, C?.2, C?.2, C?.2, C?.2, C?.2, J?.1 (Shield), J?.1 (Shield), U?.1 (A1), U?.2 (A0), U?.6 (GND)
- net at U?.10 (DIO2): now also RN?.5 (R4.2) (x2)
- net at U?.16 (SCK): now also RN?.8 (R1.2) (x2)
- net at U?.17 (MISO): now also RN?.7 (R2.2) (x2)
- net at U?.18 (MOSI): now also RN?.6 (R3.2) (x2)
- net at U?.19 (NSS): now also RN?.5 (R4.2) (x2)
- net at U?.2 (VR_ANA): now also C?.1 (x2)
- net at U?.4 (VR_DIG): now also C?.1 (x2)
- net at U?.7 (~{RESET}): now also RN?.8 (R1.2) (x2)
- net at U?.8 (DIO0): now also RN?.7 (R2.2) (x2)
- net at U?.9 (DIO1): now also RN?.6 (R3.2) (x2)
- new net: C?.1, Q?.4 (S), R?.2, R?.2
- new net: C?.1, R?.1, U?.8 (IN+)
- new net: C?.2, R?.2, U?.7 (IN-)
- new net PM_SCL: U?.4 (SCL)
- new net PM_SDA: U?.3 (SDA)
- new net RF_MISO: RN?.2 (R2.1), RN?.2 (R2.1)
- new net RF_MOSI: RN?.3 (R3.1), RN?.3 (R3.1)
- new net RF_SCK: RN?.1 (R1.1), RN?.1 (R1.1)
- new net UHF_DIO0: RN?.2 (R2.1)
- new net UHF_DIO1: RN?.3 (R3.1)
- new net UHF_DIO2: RN?.4 (R4.1)
- new net UHF_NSS: RN?.4 (R4.1)
- new net UHF_RESET: RN?.1 (R1.1)
- new net VHF_DIO0: RN?.2 (R2.1)
- new net VHF_DIO1: RN?.3 (R3.1)
- new net VHF_DIO2: RN?.4 (R4.1)
- new net VHF_NSS: RN?.4 (R4.1)
- new net VHF_RESET: RN?.1 (R1.1)
- no-connect marks 20 -> 28
Other:
- moved on the sheet: C?, J?, L?, SW?, U?

Commit message: Last commit before sensor changes
Parts:
- removed RN? (x4): 100, symbol Device:R_Pack04
- added C? (x3): 0.1u, symbol Device:C_Small
- added C? (x2): 1n, symbol Device:C_Small
- added C?: 22u, symbol Device:C_Small
- added FB? (x17): FerriteBead_Small, symbol Device:FerriteBead_Small
- added FB?: FB, symbol Device:FerriteBead_Small
- added L?: 1u, symbol Device:L_Small
- added Y? (x2): ECS-TXO-25CSMV-320-BM-TR, OSC_ECS-TXO-25CSMV-320-BM-TR, symbol HABParts:ECS-TXO-25CSMV-320-BM-TR
Connections:
- net +3V3: now also C?.1, C?.1, FB?.2, FB?.2, L?.2; no longer C?.1, C?.1, U?.15 (FB), U?.17 (VOUT), U?.18 (VOUT), U?.19 (VOUT), U?.20 (VOUT)
- net GND: now also C?.2, C?.2, C?.2, C?.2, Y?.1 (TRI_STATE), Y?.1 (TRI_STATE), Y?.2 (GND), Y?.2 (GND)
- net RF_MISO: now also FB?.1, FB?.1
- net RF_MOSI: now also FB?.1, FB?.1
- net RF_SCK: now also FB?.1, FB?.1
- net UHF_DIO0: now also FB?.1
- net UHF_DIO1: now also FB?.1
- net UHF_DIO2: now also FB?.1
- net UHF_NSS: now also FB?.1
- net UHF_RESET: now also FB?.1
- net VHF_DIO0: now also FB?.1
- net VHF_DIO1: now also FB?.1
- net VHF_DIO2: now also FB?.1
- net VHF_NSS: now also FB?.1
- net VHF_RESET: now also FB?.1
- net at U?.19 (NSS): now also FB?.2 (x2)
- net at U?.18 (MOSI): now also FB?.2 (x2)
- net at U?.17 (MISO): now also FB?.2 (x2)
- net at U?.16 (SCK): now also FB?.2 (x2)
- net at U?.10 (DIO2): now also FB?.2 (x2)
- net at U?.5 (XTA): now also C?.1 (x2)
- net at U?.7 (~{RESET}): now also FB?.2 (x2)
- net at U?.8 (DIO0): now also FB?.2 (x2)
- net at U?.9 (DIO1): now also FB?.2 (x2)
- new net: C?.1, C?.1, L?.1, U?.15 (FB), U?.17 (VOUT), U?.18 (VOUT), U?.19 (VOUT), U?.20 (VOUT)
- new net: C?.1, FB?.1, Y?.4 (VDD) (x2)
- new net: C?.2, Y?.3 (OUTPUT) (x2)

Commit message: Update to BME688 sensor
Parts:
- removed C? (x3): 0.1u, symbol Device:C_Small
- removed R?: 10K, symbol Device:R_Small
- removed R?: 10K (DNF), symbol Device:R_Small
- removed U?: BMP581, HABParts:BMP581, symbol HABParts:BMP581
- removed U?: ADT7410TRZ, SOIC127P600X175-8N_ADT7410TRZ, symbol HABParts:ADT7410TRZ
- added C? (x2): 0.1u, symbol Device:C_Small
- added U?: BME680, Package_LGA:Bosch_LGA-8_3x3mm_P0.8mm_ClockwisePinNumbering, symbol Sensor:BME680
Connections:
- net +3V3: now also C?.1, C?.1, U?.2 (CSB), U?.5 (SDO), U?.6 (VDDIO), U?.8 (VDD)
- net GND: now also C?.2, C?.2, U?.1 (GND), U?.7 (GND)
- new net BME_SCL: U?.4 (SCK)
- new net BME_SDA: U?.3 (SDI)

Commit message: USB Mux Addition
Parts:
- added C?: 0.1u, symbol Device:C_Small
- added J?: USB_C_Receptacle_USB2.0, symbol Connector:USB_C_Receptacle_USB2.0
- added R? (x2): 5.1K, symbol Device:R_Small
- added R? (x2): 27.4, symbol Device:R_Small
- added R? (x2): 2.2K, symbol Device:R_Small
- added SW?: MCU/GNSS USB, symbol Switch:SW_SPDT
- added U?: USB3740B-AI9, Package_DFN_QFN:UQFN-10_1.6x2.1mm_P0.5mm, symbol Interface_USB:USB3740B-AI9
Connections:
- net GNSS_SCL is gone; now on net BME_SCL: U?.19 (SCL/SPI_CLK)
- net GNSS_SDA is gone; now on net BME_SDA: U?.18 (SDA/SPI_CS_N)
- net IMU_SCL is gone; now on net BME_SCL: U?.11 (B2)
- net IMU_SDA is gone; now on net BME_SDA: U?.10 (B1)
- net PM_SCL is gone; now on net BME_SCL: U?.4 (SCL)
- net PM_SDA is gone; now on net BME_SDA: U?.3 (SDA)
- net +3V3: now also C?.1, R?.2, R?.2, SW?.3 (C), U?.5 (VDD)
- net BME_SCL: now also U?.7 (GPIO5), R?.1
- net BME_SDA: now also U?.6 (GPIO4), R?.1
- net GND: now also C?.2, J?.A1 (GND), J?.A12 (GND), J?.B1 (GND), J?.B12 (GND), J?.S1 (SHIELD), R?.1, R?.2, SW?.1 (A), U?.3 (OE_N), U?.8 (GND); no longer U?.7 (V_USB)
- net RF_MISO: now also U?.27 (GPIO16)
- net RF_MOSI: now also U?.30 (GPIO19)
- net RF_SCK: now also U?.29 (GPIO18)
- net at U?.5 (USB_DM): now also R?.1
- net at U?.6 (USB_DP): now also R?.1
- net DN renamed MCU_USBM
- net MCU_USBM: now also U?.1 (DM_1)
- net DP renamed MCU_USBP
- net MCU_USBP: now also U?.2 (DP_1)
- new net: J?.A5 (CC1), R?.1
- new net: J?.B5 (CC2), R?.2
- new net: SW?.2 (B), U?.4 (S), U?.7 (V_USB)
- new net: J?.A6 (D+), J?.B6 (D+), U?.10 (DP)
- new net: J?.A7 (D-), J?.B7 (D-), U?.9 (DM)
- new net: J?.A4 (VBUS), J?.A9 (VBUS), J?.B4 (VBUS), J?.B9 (VBUS)
- new net GNSS_USBM: R?.2, U?.7 (DM_2)
- new net GNSS_USBP: R?.2, U?.6 (DP_2)
Other:
- moved on the sheet: C?, FB?, J?, L?, U?, Y?
