File: HABBoard/HABBoard.kicad_sch (KiCad schematic)
At the start: 154 parts

Commit message: Added Power Switch IC, more filtering, and other stuff
Parts:
- removed C?: 0.1u, symbol Device:C_Small
- removed J?: SWD, symbol Connector:Conn_01x03_Male
- removed SW?: RESET, symbol Switch:SW_Push
- removed SW?: MCU/GNSS USB, symbol Switch:SW_SPDT
- removed U?: USB3740B-AI9, Package_DFN_QFN:UQFN-10_1.6x2.1mm_P0.5mm, symbol Interface_USB:USB3740B-AI9
- added C? (x6): 1u, symbol Device:C_Small
- added C? (x5): 0.1u, symbol Device:C_Small
- added C? (x2): 47u, symbol Device:C_Polarized_Small
- added C?: 22u, symbol Device:C_Small
- added C?: 10u, symbol Device:C_Small
- added D? (x2): SP0503BAHT, Package_TO_SOT_SMD:SOT-143, symbol Power_Protection:SP0503BAHT
- added J?: MEM2067-02-180-00-A_REVB, HABParts:GCT_MEM2067-02-180-00-A_REVB, symbol HABParts:MEM2067-02-180-00-A_REVB
- added J?: DEBUG, symbol Connector:Conn_01x05_Male
- added J?: USB_C_MCU, symbol Connector:USB_C_Receptacle_USB2.0
- added J?: GNSS_UART, symbol Connector:Conn_01x03_Male
- added L?: 1u, symbol Device:L_Small
- added R? (x2): 5.1K, symbol Device:R_Small
- added R?: 220k, symbol Device:R_Small
- added R?: 100K, symbol Device:R_Small
- added R?: 100k, symbol Device:R_Small
- added TP?: GNSS_RESET, symbol Connector:TestPoint
- added U?: TC2015-3.3VxCTTR, Package_TO_SOT_SMD:SOT-23-5, symbol Regulator_Linear:TC2015-3.3VxCTTR
- added U?: TPS2116DRLR, HABParts:SOTFL50P160X60-8N, symbol HABParts:TPS2116DRLR
- C? (x4): value 2.2u -> 1u
- C?: value 10u -> 1u
- J?: value USB_C_Receptacle_USB2.0 -> USB_C_GNSS
Connections:
- net GNSS_USBM is gone; now on an unnamed net: R?.2
- net GNSS_USBP is gone; now on an unnamed net: R?.2
- net +3V3: now also C?.1, C?.1, C?.1, C?.1, C?.1, C?.1, C?.1, J?.4 (VDD), L?.2, U?.3 (ON/~{OFF}); no longer C?.1, C?.1, L?.2, U?.1 (IOVDD), U?.10 (IOVDD), U?.22 (IOVDD), U?.33 (IOVDD), U?.42 (IOVDD), U?.49 (IOVDD)
- net +SYS: now also C?.1, C?.1
- net GND: now also C?.1, C?.2, C?.2, C?.2, C?.2, C?.2, C?.2, C?.2, C?.2, C?.2, C?.2, C?.2, C?.2, C?.2, C?.2, D?.1 (A), D?.1 (A), J?.10 (SHIELD), J?.11 (SHIELD), J?.12 (SHIELD), J?.3 (Pin_3), J?.5 (Pin_5), J?.6 (VSS), J?.9 (SHIELD), J?.A1 (GND), J?.A12 (GND), J?.B1 (GND), J?.B12 (GND), J?.S1 (SHIELD), R?.1, R?.1, R?.2, R?.2, U?.1 (GND), U?.2 (GND); no longer U?.52 (QSPI_SCLK), U?.6 (CLK)
- net IMU_INT: now also U?.36 (GPIO24)
- net UHF_DIO0: now also U?.31 (GPIO20)
- net UHF_DIO1: now also U?.32 (GPIO21)
- net UHF_DIO2: now also U?.34 (GPIO22)
- net UHF_NSS: now also U?.12 (GPIO9)
- net UHF_RESET: now also U?.9 (GPIO7)
- net VHF_DIO0: now also U?.17 (GPIO14)
- net VHF_DIO1: now also U?.18 (GPIO15)
- net VHF_DIO2: now also U?.28 (GPIO17)
- net VHF_NSS: now also U?.11 (GPIO8)
- net VHF_RESET: now also U?.8 (GPIO6)
- net at C?.1, U?.2 (VOUT), U?.22 (V_BCKP): now also C?.1
- net MCU_BOOT: now reaches R?.1, SW?.2
- net MCU_BOOT: now also J?.3 (Pin_3)
- net at C?.1, C?.1, L?.1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: now also C?.1
- net at C?.1, Q?.4 (S): now also U?.6 (IN2); no longer R?.2, R?.2
- net at U?.24 (SWCLK): now also J?.1 (Pin_1)
- net at U?.25 (SWD): now also J?.2 (Pin_2)
- net at U?.20 (TXD/SPI_MISO): now also J?.1 (Pin_1)
- net at U?.21 (RXD/SPI_MOSI): now also J?.2 (Pin_2)
- net GNSS_TP: now reaches U?.3 (TIMEPULSE)
- net GNSS_TXR: now reaches U?.4 (EXTINT)
- net GNSS_TXR: now also U?.35 (GPIO23)
- net at U?.7 (V_USB): now also C?.1, C?.1, R?.1, U?.5 (VOUT)
- net at U?.8 (RESET_N): now also TP?.1
- net MCU_RESET: now reaches SW?.2, U?.26 (RUN)
- net MCU_RESET: now also J?.4 (Pin_4)
- net SMPS_MODE: now reaches U?.12 (MODE)
- net SD_SCK: now reaches U?.13 (GPIO10)
- net SD_SCK: now also J?.5 (CLK)
- net SD_MOSI: now reaches U?.14 (GPIO11)
- net SD_MOSI: now also J?.3 (CMD)
- net SD_MISO: now reaches U?.15 (GPIO12)
- net SD_MISO: now also J?.7 (DAT0)
- net SD_CS: now reaches U?.16 (GPIO13)
- net SD_CS: now also J?.2 (CD/DAT3)
- net at J?.A6 (D+), J?.B6 (D+): now also D?.4 (K)
- net at J?.A7 (D-), J?.B7 (D-): now also D?.3 (K)
- net at J?.A4 (VBUS), J?.A9 (VBUS), J?.B4 (VBUS)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: now also C?.2, D?.2 (K), U?.1 (VIN)
- net MCU_USBM: no longer names the net of R?.2
- net MCU_USBM: now also D?.3 (K), J?.A7 (D-), J?.B7 (D-)
- net MCU_USBP: no longer names the net of R?.2
- net MCU_USBP: now also D?.4 (K), J?.A6 (D+), J?.B6 (D+)
- new net: C?.1, C?.1, L?.1, L?.2
- new net: U?.52 (QSPI_SCLK), U?.6 (CLK)
- new net: R?.2, R?.2, U?.2 (OUT), U?.7 (OUT)
- new net: R?.1, R?.2, U?.4 (PR1)
- new net: J?.B5 (CC2), R?.2
- new net: J?.A5 (CC1), R?.1
- new net: U?.1 (IOVDD), U?.10 (IOVDD), U?.22 (IOVDD), U?.33 (IOVDD), U?.42 (IOVDD), U?.49 (IOVDD)
- new net USB_VBUS: C?.1, D?.2 (K), J?.A4 (VBUS), J?.A9 (VBUS), J?.B4 (VBUS), J?.B9 (VBUS), R?.2, U?.3 (IN1), U?.5 (MODE)
- no-connect marks 28 -> 33
Other:
- moved on the sheet: BT?, C?, FB?, J?, L?, Q?, R?, SW?, TP?, U?, Y?

Commit message: Final Schematic v1
Parts:
- added D?: VHF_TX, symbol Device:LED
- added D?: GNSS_STATUS, symbol Device:LED_Dual_AAKK
- added D?: MCU_HEARTBEAT, symbol Device:LED
- added D?: UHF_STATUS, symbol Device:LED_Dual_AAKK
- added Q? (x6): SSM6N7002KFU, Package_TO_SOT_SMD:SOT-363_SC-70-6, symbol HABParts:SSM6N7002KFU
- added R? (x12): 220, symbol Device:R_Small
- added SW?: USER_BUTTON, symbol Switch:SW_Push
Connections:
- net +3V3: now also D?.1 (A1), D?.1 (A1), D?.2 (A), D?.2 (A), D?.2 (A2), D?.2 (A2)
- net GND: now also Q?.1 (S), Q?.1 (S), Q?.1 (S), Q?.4 (S), Q?.4 (S), Q?.4 (S), SW?.1
- net GNSS_TP: now also U?.37 (GPIO25)
- net SMPS_MODE: now also U?.38 (GPIO26_ADC0)
- net GNSS_SGRN: now reaches U?.2 (GPIO0)
- net GNSS_SGRN: now also R?.2
- net GNSS_SRED: now reaches U?.3 (GPIO1)
- net GNSS_SRED: now also R?.2
- net VHF_SGRN: now reaches U?.39 (GPIO27_ADC1)
- net VHF_SGRN: now also R?.2
- net UHF_SGRN: now reaches U?.4 (GPIO2)
- net UHF_SGRN: now also R?.2
- net MCU_HB: now reaches U?.40 (GPIO28_ADC2)
- net MCU_HB: now also R?.2
- net at U?.41 (GPIO29_ADC3): now also SW?.2
- net UHF_SRED: now reaches U?.5 (GPIO3)
- net UHF_SRED: now also R?.2
- new net: Q?.3 (D), R?.2 (x3)
- new net: Q?.5 (G), R?.1 (x3)
- new net: D?.3 (K1), R?.1 (x2)
- new net: Q?.2 (G), R?.1 (x3)
- new net: Q?.6 (D), R?.1 (x3)
- new net: D?.4 (K2), R?.2 (x2)
- new net: D?.1 (K), R?.1
- new net: D?.1 (K), R?.2
Other:
- moved on the sheet: R?

Commit message: Final Schematic v2, begin footprint addition
Parts:
- added C39: 0.1u, Capacitor_SMD:C_0402_1005Metric, symbol Device:C_Small
- added H1, H2, H3, H4: MountingHole_Pad, symbol Mechanical:MountingHole_Pad
- added TP1: GND, TestPoint:TestPoint_Pad_D1.0mm, symbol Connector:TestPoint
- added TP10: VSYS, TestPoint:TestPoint_Pad_D1.0mm, symbol Connector:TestPoint
- added TP11: VMAIN, TestPoint:TestPoint_Pad_D1.0mm, symbol Connector:TestPoint
- added TP2: VUSB_GNSS, TestPoint:TestPoint_Pad_D1.0mm, symbol Connector:TestPoint
- added TP5: VRTC, TestPoint:TestPoint_Pad_D1.0mm, symbol Connector:TestPoint
- added TP6: VCORE, TestPoint:TestPoint_Pad_D1.0mm, symbol Connector:TestPoint
- added TP7: VIMU, TestPoint:TestPoint_Pad_D1.0mm, symbol Connector:TestPoint
- added TP8: VBATT, TestPoint:TestPoint_Pad_D1.0mm, symbol Connector:TestPoint
- added TP9: VUSB, TestPoint:TestPoint_Pad_D1.0mm, symbol Connector:TestPoint
- C1, C10, C11, C12, C13, C14, C15, C16, C17, C18, C19, C2, C20, C21, C22, C23, C24, C25, C26, C27, C28, C29, C3, C30, C31, C32, C33, C34, C35, C36, C37, C4, C40, C41, C42, C43, C44, C45, C46, C47, C48, C49, C5, C50, C51, C52, C53, C54, C55, C56, C57, C58, C59, C6, C60, C61, C62, C63, C64, C65, C66, C67, C68, C69, C7, C70, C71, C72, C73, C74, C76, C77, C78, C79, C8, C86, C9: renamed from C?; footprint (none) -> Capacitor_SMD:C_0402_1005Metric
- C38: renamed from C?; value C -> 0.1u; footprint (none) -> Capacitor_SMD:C_0402_1005Metric
- C80: renamed from C?; value 10u -> 22u
- J1, J2: renamed from J?; footprint (none) -> Connector_USB:USB_C_Receptacle_GCT_USB4085
- J7: renamed from J?; footprint (none) -> Connector_PinHeader_2.54mm:PinHeader_1x03_P2.54mm_Vertical
- J8: renamed from J?; footprint (none) -> Connector_PinHeader_2.54mm:PinHeader_1x05_P2.54mm_Vertical
- L1, L10, L2, L3, L4, L5, L6, L7, L8, L9: renamed from L?; footprint (none) -> Inductor_SMD:L_0402_1005Metric
- R36, R37: renamed from R?; value R -> 22
- SW4: renamed from SW?; footprint (none) -> TestPoint:TestPoint_Pad_D1.0mm
- TP3, TP4: renamed from TP?; footprint (none) -> TestPoint:TestPoint_Pad_D1.0mm
- Y1: renamed from Y?; footprint (none) -> HABParts:445C25D12M00000
- Y2: renamed from Y?; footprint OSC_ECS-TXO-25CSMV-320-BM-TR -> HABParts:OSC_ECS-TXO-25CSMV-320-BM-TR
- Y3: renamed from Y?; footprint OSC_ECS-TXO-25CSMV-320-BM-TR -> TestPoint:TestPoint_Pad_D1.0mm
- gave numbers to parts that had none: 98
Connections:
- net +1V1: now also TP6.1
- net +1V8: now also TP7.1
- net +3V3: now also U1.1 (IOVDD), U1.10 (IOVDD), U1.22 (IOVDD), U1.33 (IOVDD), U1.42 (IOVDD), U1.49 (IOVDD), U13.6 (VDD), C39.1, TP11.1
- net +SYS: now also TP10.1
- net GND: now also C39.2, TP1.1; no longer J1.S1 (SHIELD), J2.S1 (SHIELD)
- net USB_VBUS: now also TP9.1
- net at C46.1, C47.1, U2.22 (V_BCKP)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: now also TP5.1
- net at C52.1, Q4.4 (S), U15.6 (IN2): now also TP8.1
- net at C43.1, C44.1, R10.1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: now also TP2.1
- no-connect marks 33 -> 35

Commit message: Adding Reference Designators, again...
Parts:
- C62: renamed from C54; footprint Capacitor_SMD:C_0402_1005Metric -> (none)
- C63: renamed from C55; footprint Capacitor_SMD:C_0402_1005Metric -> (none)
- C64: renamed from C69; footprint Capacitor_SMD:C_0402_1005Metric -> (none)
- C66: renamed from C60; footprint Capacitor_SMD:C_0402_1005Metric -> (none)
- C67: renamed from C58; footprint Capacitor_SMD:C_0402_1005Metric -> (none)
- C68: renamed from C63; footprint Capacitor_SMD:C_0402_1005Metric -> (none)
- C69: renamed from C61; footprint Capacitor_SMD:C_0402_1005Metric -> (none)
- C70: renamed from C67; footprint Capacitor_SMD:C_0402_1005Metric -> (none)
- C71: renamed from C74; footprint Capacitor_SMD:C_0402_1005Metric -> (none)
- C73: renamed from C65; footprint Capacitor_SMD:C_0402_1005Metric -> (none)
- C75: renamed from C59; footprint Capacitor_SMD:C_0402_1005Metric -> (none)
- C76: renamed from C64; footprint Capacitor_SMD:C_0402_1005Metric -> (none)
- C77: renamed from C71; footprint Capacitor_SMD:C_0402_1005Metric -> (none)
- C78: renamed from C62; footprint Capacitor_SMD:C_0402_1005Metric -> (none)
- C79: renamed from C73; footprint Capacitor_SMD:C_0402_1005Metric -> (none)
- C80: renamed from C68; footprint Capacitor_SMD:C_0402_1005Metric -> (none)
- C81: renamed from C66; footprint Capacitor_SMD:C_0402_1005Metric -> (none)
- C82: renamed from C70; footprint Capacitor_SMD:C_0402_1005Metric -> (none)
- C84: renamed from C72; footprint Capacitor_SMD:C_0402_1005Metric -> (none)
- C85: renamed from C56; footprint Capacitor_SMD:C_0402_1005Metric -> (none)
- C86: renamed from C57; footprint Capacitor_SMD:C_0402_1005Metric -> (none)
- renumbered BT1 to BT?, C19 to C15, C20 to C16, C21 to C17, C22 to C18, C23 to C19, C24 to C20, C25 to C21, C26 to C22, C39 to C23, C27 to C24, C28 to C25, C29 to C26, C30 to C27, C31 to C28, C32 to C29, C33 to C30, C34 to C31, C35 to C32, C36 to C33, C37 to C34, C15 to C35, C16 to C36, C17 to C37, C18 to C38, C38 to C39, C86 to C40, C40 to C41, C41 to C42, C42 to C43, C43 to C44, C44 to C45, C45 to C46, C46 to C47, C47 to C48, C48 to C49, C49 to C50, C50 to C51, C51 to C52, C52 to C53, C53 to C54, C80 to C55, C81 to C56, C82 to C57, C83 to C58, C85 to C59, C75 to C60, C84 to C61, C78 to C65, C77 to C72, C79 to C74, C76 to C83, D6 to D?, D1 to D?, D3 to D?, D2 to D?, D5 to D?, D4 to D?, FB2 to FB?, FB17 to FB?, FB16 to FB?, FB12 to FB?, FB13 to FB?, FB6 to FB?, FB14 to FB?, FB8 to FB?, FB4 to FB?, FB10 to FB?, FB11 to FB?, FB15 to FB?, FB18 to FB?, FB3 to FB?, FB9 to FB?, FB1 to FB?, FB7 to FB?, FB5 to FB?, H1 to H?, H3 to H?, H2 to H?, H4 to H?, J2 to J1, J1 to J2, J5 to J?, J4 to J?, J6 to J?, J8 to J?, J9 to J?, J10 to J?, J7 to J?, J3 to J?, L1 to L?, L5 to L?, L8 to L?, L7 to L?, L6 to L?, L11 to L?, L10 to L?, L9 to L?, L3 to L?, L13 to L?, L12 to L?, L2 to L?, L4 to L?, Q2 to Q?, Q1 to Q?, Q3 to Q?, Q4 to Q?, R5 to R?, R12 to R?, R13 to R?, R17 to R?, R22 to R?, R31 to R?, R2 to R?, R8 to R?, R20 to R?, R24 to R?, R25 to R?, R27 to R?, R29 to R?, R18 to R?, R1 to R?, R36 to R?, R16 to R?, R6 to R?, R35 to R?, R11 to R?, R28 to R?, R14 to R?, R15 to R?, R21 to R?, R3 to R?, R4 to R?, R26 to R?, R33 to R?, R30 to R?, R19 to R?, R23 to R?, R10 to R?, R9 to R?, R7 to R?, R32 to R?, R37 to R?, R34 to R?, SW4 to SW?, TP7 to TP?, TP10 to TP?, TP5 to TP?, TP1 to TP?, TP8 to TP?, TP4 to TP?, TP11 to TP?, TP9 to TP?, TP2 to TP?, TP3 to TP?, TP6 to TP?, U6 to U1, U4 to U10, U5 to U11, U7 to U2, U2 to U3, U8 to U4, U1 to U5, U9 to U6, U10 to U7, U3 to U8, U11 to U9, Y2 to Y1, Y3 to Y2, Y1 to Y3
Connections:
- no-connect marks 35 -> 39
Other:
- moved on the sheet: H?
