File: HABBoard/HABBoard.kicad_sch (KiCad schematic)
At the start: 216 parts, among them J1 USB_C_GNSS, J2 USB_C_MCU, SW1 RESET, SW2 BOOT, SW3 USER_BUTTON, U1 TC2015-3.3VxCTTR, U10 SX1276, U11 SX1276, U12 MP5016GQH-Z, U13 PE42421, U14 ISL91127IR, U15 TPS2116DRLR, U16 INA219BxD, U2 W25Q128JVS, U3 NEO-M9N-00B, U4 AP2138N-2.5, U5 RP2040, U6 BME680, U7 TXS0104E, U8 ICM-20948, U9 AP2138N-1.8, Y1 ECS-TXO-25CSMV-320-BM-TR, Y2 ECS-TXO-25CSMV-320-BM-TR, Y3 12.000MHz

Commit message: Schematic Annotation
Parts:
- removed SW?: Power, TestPoint:TestPoint_Pad_D1.0mm, symbol Switch:SW_SPST
- added SW4: Power, symbol Switch:SW_SPDT
- gave numbers to parts that had none: 102
- renumbered J2 to J1, J1 to J2
Connections:
- net +SYS: now also SW4.1 (A)
- net at U14.11 (EN): now also SW4.2 (B)
- no-connect marks 39 -> 40

Commit message: Mostly finished footprint association
Parts:
- C40, C41, C42, C43, C44, C45, C46, C47, C48, C49, C50, C51, C52, C53, C54: footprint Capacitor_SMD:C_0402_1005Metric -> Capacitor_SMD:C_0603_1608Metric
- C55, C56, C57, C58, C59: footprint (none) -> Capacitor_SMD:C_0805_2012Metric
- C60, C61: footprint (none) -> Capacitor_SMD:CP_Elec_5x5.3
- C62, C63, C64, C66, C67, C68, C69, C70, C71, C73, C75, C76, C77, C78, C79, C80, C81, C82, C84, C85, C86: footprint (none) -> Capacitor_SMD:C_0402_1005Metric
- D5, D6: footprint (none) -> LED_SMD:LED_0603_1608Metric
- FB1, FB10, FB11, FB12, FB13, FB14, FB15, FB16, FB17, FB18, FB2, FB3, FB4, FB5, FB6, FB7, FB8, FB9: footprint (none) -> Inductor_SMD:L_0402_1005Metric
- H1, H2, H3, H4: footprint (none) -> MountingHole:MountingHole_3.2mm_M3_Pad
- R1, R10, R11, R12, R13, R14, R15, R16, R17, R18, R19, R2, R20, R21, R22, R23, R24, R25, R26, R27, R28, R29, R3, R30, R31, R32, R33, R34, R35, R36, R4, R5, R6, R7, R8, R9: footprint (none) -> Resistor_SMD:R_0402_1005Metric
- R37: footprint (none) -> Resistor_SMD:R_1206_3216Metric
- SW1, SW2, SW3: footprint (none) -> HABParts:PTS815SJK250SMTRLFS
- SW4: footprint (none) -> HABParts:SW_JS102011SCQN

Commit message: Footprint assignment complete
Parts:
- removed J10, J9: RFShield_TwoPieces, symbol Device:RFShield_TwoPieces
- removed J4: GPS_SMA, symbol Connector:Conn_Coaxial
- removed J7: 144MHz, symbol Connector:Conn_Coaxial
- removed J8: 915MHz, symbol Connector:Conn_Coaxial
- added J4: GPS In, HABParts:LPRS_SMA_CONNECTOR, symbol HABParts:LPRS_SMA
- added J7: VHF Out, HABParts:LPRS_SMA_CONNECTOR, symbol HABParts:LPRS_SMA
- added J8: UHF Out, HABParts:LPRS_SMA_CONNECTOR, symbol HABParts:LPRS_SMA
- BT1: footprint (none) -> HABParts:CUI_TB002-500-02BE
- D3, D4: footprint (none) -> LED_SMD:LED_RGB_Wuerth-PLCC4_3.2x2.8mm_150141M173100
- L1, L2, L3: footprint (none) -> Inductor_SMD:L_Coilcraft_XxL4020
Connections:
- net GND: now also J4.1 (In), J7.G1 (Ext), J7.G2 (Ext), J7.G3 (Ext), J7.G4 (Ext), J8.G1 (Ext), J8.G2 (Ext), J8.G3 (Ext), J8.G4 (Ext)
- net at L4.2, U3.11 (RF_IN): now also J4.G1 (Ext), J4.G2 (Ext), J4.G3 (Ext), J4.G4 (Ext)
- net at C65.1, L8.2: now also J7.1 (In)
- net at C74.2: now also J8.1 (In)

Commit message: Initial PCB Layout
Parts:
- U12: footprint HABParts:IC_MP5016GQH-Z -> HABParts:MP5016GQH-Z
Changed lines of the file:
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@@
     (property "Reference" "U12" (id 0) (at 407.797 35.052 0))
     (property "Value" "MP5016GQH-Z" (id 1) (at 407.797 37.592 0))
-    (property "Footprint" "HABParts:IC_MP5016GQH-Z" (id 2) (at 407.797 53.594 0)
+    (property "Footprint" "HABParts:MP5016GQH-Z" (id 2) (at 407.797 53.594 0)
       (effects (font (size 1.27 1.27)) (justify bottom) hide)
     )
@@
     )
     (path "/5d049acd-4e60-480d-9511-dd18a2d5ceee"
-      (reference "U12") (unit 1) (value "MP5016GQH-Z") (footprint "HABParts:IC_MP5016GQH-Z")
+      (reference "U12") (unit 1) (value "MP5016GQH-Z") (footprint "HABParts:MP5016GQH-Z")
     )
     (path "/78200126-0dac-4eb0-861b-cf1ffb0904f6"

Commit message: PCB Layout Work
Parts:
- Y2: footprint TestPoint:TestPoint_Pad_D1.0mm -> HABParts:OSC_ECS-TXO-25CSMV-320-BM-TR
Connections:
- net GND: now also J4.G1 (Ext), J4.G2 (Ext), J4.G3 (Ext), J4.G4 (Ext); no longer J4.1 (In)
- new net: J4.1 (In), L4.2, U3.11 (RF_IN)
Other:
- moved on the sheet: J4
Changed lines of the file:
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@@
     (property "Reference" "Y2" (id 0) (at 306.197 293.497 0))
     (property "Value" "ECS-TXO-25CSMV-320-BM-TR" (id 1) (at 306.197 296.037 0))
-    (property "Footprint" "TestPoint:TestPoint_Pad_D1.0mm" (id 2) (at 306.197 306.197 0)
+    (property "Footprint" "HABParts:OSC_ECS-TXO-25CSMV-320-BM-TR" (id 2) (at 306.197 306.197 0)
       (effects (font (size 1.27 1.27)) (justify bottom) hide)
     )
@@
     (pin "4")
   )
-  (symbol (lib_id "HABParts:LPRS_SMA") (at 75.184 231.394 90) (unit 1)
+  (symbol (lib_id "HABParts:LPRS_SMA") (at 75.184 231.394 0) (mirror y) (unit 1)
     (in_bom yes) (on_board yes) (fields_autoplaced)
-    (property "Reference" "J4" (id 0) (at 75.4772 224.536 90))
-    (property "Value" "GPS In" (id 1) (at 75.4772 227.076 90))
-    (property "Footprint" "HABParts:LPRS_SMA_CONNECTOR" (id 2) (at 67.564 231.394 0)
+    (property "Reference" "J4" (id 0) (at 75.5014 224.79 0))
+    (property "Value" "GPS In" (id 1) (at 75.5014 227.33 0))
+    (property "Footprint" "HABParts:LPRS_SMA_CONNECTOR" (id 2) (at 75.184 223.774 0)
       (effects (font (size 1.27 1.27)) hide)
     )
-    (property "Datasheet" "https://www.mouser.com/datasheet/2/743/LPRS_04102019_SMAconnector-1568179.pdf" (id 3) (at 65.024 246.634 0)
+    (property "Datasheet" "https://www.mouser.com/datasheet/2/743/LPRS_04102019_SMAconnector-1568179.pdf" (id 3) (at 90.424 221.234 0)
       (effects (font (size 1.27 1.27)) hide)
     )
@@
     )
     (path "/637c10f8-2d33-43d4-a8ad-f8b48bc2f43b"
-      (reference "Y2") (unit 1) (value "ECS-TXO-25CSMV-320-BM-TR") (footprint "TestPoint:TestPoint_Pad_D1.0mm")
+      (reference "Y2") (unit 1) (value "ECS-TXO-25CSMV-320-BM-TR") (footprint "HABParts:OSC_ECS-TXO-25CSMV-320-BM-TR")
     )
     (path "/88a3639d-9ebc-4ea6-bee9-327c94a642ae"

Commit message: More Routing
Parts:
- added J10, J9: RFShield_TwoPieces, HABParts:SMS409F, symbol Device:RFShield_TwoPieces
Connections:
- net GND: now also J10.1 (Shield), J9.1 (Shield)
Changed lines of the file:
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@@
     (pin "2")
   )
+  (symbol (lib_id "power:GND") (at 543.306 248.412 0) (unit 1)
+    (in_bom yes) (on_board yes) (fields_autoplaced)
+    (property "Reference" "#PWR01" (id 0) (at 543.306 254.762 0)
+      (effects (font (size 1.27 1.27)) hide)
+    )
+    (property "Value" "GND" (id 1) (at 543.306 253.492 0))
+    (property "Footprint" "" (id 2) (at 543.306 248.412 0)
+      (effects (font (size 1.27 1.27)) hide)
+    )
+    (property "Datasheet" "" (id 3) (at 543.306 248.412 0)
+      (effects (font (size 1.27 1.27)) hide)
+    )
+    (pin "1")
+  )
   (symbol (lib_id "power:GND") (at 408.432 320.167 0) (unit 1)
     (in_bom yes) (on_board yes) (fields_autoplaced)
@@
     (pin "1")
   )
+  (symbol (lib_id "power:GND") (at 543.306 274.828 0) (unit 1)
+    (in_bom yes) (on_board yes) (fields_autoplaced)
+    (property "Reference" "#PWR02" (id 0) (at 543.306 281.178 0)
+      (effects (font (size 1.27 1.27)) hide)
+    )
+    (property "Value" "GND" (id 1) (at 543.306 279.908 0))
+    (property "Footprint" "" (id 2) (at 543.306 274.828 0)
+      (effects (font (size 1.27 1.27)) hide)
+    )
+    (property "Datasheet" "" (id 3) (at 543.306 274.828 0)
+      (effects (font (size 1.27 1.27)) hide)
+    )
+    (pin "1")
+  )
   (symbol (lib_id "Device:R_Small") (at 90.424 55.372 270) (unit 1)
     (in_bom yes) (on_board yes)
@@
     (pin "1")
   )
+  (symbol (lib_id "Device:RFShield_TwoPieces") (at 543.306 264.668 0) (unit 1)
+    (in_bom yes) (on_board yes) (fields_autoplaced)
+    (property "Reference" "J10" (id 0) (at 562.61 261.4929 0)
+      (effects (font (size 1.27 1.27)) (justify left))
+    )
+    (property "Value" "RFShield_TwoPieces" (id 1) (at 562.61 264.0329 0)
+      (effects (font (size 1.27 1.27)) (justify left))
+    )
+    (property "Footprint" "HABParts:SMS409F" (id 2) (at 543.306 267.208 0)
+      (effects (font (size 1.27 1.27)) hide)
+    )
+    (property "Datasheet" "~" (id 3) (at 543.306 267.208 0)
+      (effects (font (size 1.27 1.27)) hide)
+    )
+    (pin "1")
+  )
   (symbol (lib_id "Device:R_Small") (at 232.156 338.836 270) (unit 1)
     (in_bom yes) (on_board yes) (fields_autoplaced)
@@
     (pin "9")
   )
+  (symbol (lib_id "Device:RFShield_TwoPieces") (at 543.306 238.252 0) (unit 1)
+    (in_bom yes) (on_board yes) (fields_autoplaced)
+    (property "Reference" "J9" (id 0) (at 562.61 235.0769 0)
+      (effects (font (size 1.27 1.27)) (justify left))
+    )
+    (property "Value" "RFShield_TwoPieces" (id 1) (at 562.61 237.6169 0)
+      (effects (font (size 1.27 1.27)) (justify left))
+    )
+    (property "Footprint" "HABParts:SMS409F" (id 2) (at 543.306 240.792 0)
+      (effects (font (size 1.27 1.27)) hide)
+    )
+    (property "Datasheet" "~" (id 3) (at 543.306 240.792 0)
+      (effects (font (size 1.27 1.27)) hide)
+    )
+    (pin "1")
+  )
   (symbol (lib_id "Device:C_Small") (at 435.102 113.792 0) (mirror y) (unit 1)
     (in_bom yes) (on_board yes) (fields_autoplaced)
@@
   )
   (symbol_instances
+    (path "/04ca017d-b69a-4117-a209-3f98744cdfc1"
+      (reference "#PWR01") (unit 1) (value "GND") (footprint "")
+    )
+    (path "/0b431e8c-00d5-46df-a843-96f45021274e"
+      (reference "#PWR02") (unit 1) (value "GND") (footprint "")
+    )
     (path "/21ac41d7-d682-4d97-b057-a61454bc9ed3"
       (reference "#PWR0101") (unit 1) (value "GND") (footprint "")
@@
       (reference "J8") (unit 1) (value "UHF Out") (footprint "HABParts:LPRS_SMA_CONNECTOR")
     )
+    (path "/855b6ed8-9d25-4bbd-a886-72bba3c08aa4"
+      (reference "J9") (unit 1) (value "RFShield_TwoPieces") (footprint "HABParts:SMS409F")
+    )
+    (path "/4a1d8bb5-357b-42e0-b28a-e8a45b458c5c"
+      (reference "J10") (unit 1) (value "RFShield_TwoPieces") (footprint "HABParts:SMS409F")
+    )
     (path "/52fd6ae6-67d9-43eb-8b9e-7a1911b0b41a"

Commit message: Even more layout
Parts:
- removed C45: 1u, Capacitor_SMD:C_0603_1608Metric, symbol Device:C_Small
- removed J10, J9: RFShield_TwoPieces, HABParts:SMS409F, symbol Device:RFShield_TwoPieces
- removed TP6: VCORE, TestPoint:TestPoint_Pad_D1.0mm, symbol Connector:TestPoint
- added C87: 0.1u, Capacitor_SMD:C_0402_1005Metric, symbol Device:C_Small
- added J10, J9: RFShield_TwoPieces, HABParts:SMS409F, symbol HABParts:RFShield_TwoPieces
Connections:
- net +1V8: now also C87.1
- net GND: now also C87.2, J10.1 (Shield), J10.10 (Shield), J10.11 (Shield), J10.12 (Shield), J10.13 (Shield), J10.14 (Shield), J10.15 (Shield), J10.16 (Shield), J10.2 (Shield), J10.3 (Shield), J10.4 (Shield), J10.5 (Shield), J10.6 (Shield), J10.7 (Shield), J10.8 (Shield), J10.9 (Shield), J9.1 (Shield), J9.10 (Shield), J9.11 (Shield), J9.12 (Shield), J9.13 (Shield), J9.14 (Shield), J9.15 (Shield), J9.16 (Shield), J9.2 (Shield), J9.3 (Shield), J9.4 (Shield), J9.5 (Shield), J9.6 (Shield), J9.7 (Shield), J9.8 (Shield), J9.9 (Shield)

Commit message: Finish majority of routing
Parts:
- removed C7: 0.1u, Capacitor_SMD:C_0402_1005Metric, symbol Device:C_Small
- added R38: 10k, Resistor_SMD:R_0402_1005Metric, symbol Device:R_Small
Connections:
- net +3V3: now also R38.1
- net SMPS_MODE: now also R38.2
Other:
- moved on the sheet: C10, C11, C12, C8, C9
